File: 32u4 sumo deneme kartı v1.1/32u4 denemesi.brd (EAGLE design)
At the start: 100 x 100 mm, 136 parts, among them IC1 IC_555-SOIC8, IC2 LM2577S, IC3 LMV358MX, J1 AVR_SPI_PRG_6NS, Q2 SI3456BDVSOT-5-6, U1 TB6612FNG

Commit message: sws
Routing:
- net +5V: track 618.1 -> 621.9 mm
Changed lines of the file:
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@@
 <contactref element="C35" pad="1"/>
 <contactref element="C36" pad="1"/>
-<wire x1="24.384" y1="43.2816" x2="24.384" y2="47.3964" width="0.4064" layer="1"/>
+<wire x1="24.384" y1="43.2816" x2="24.384" y2="49.3964" width="0.4064" layer="1"/>
 <wire x1="24.2316" y1="43.1292" x2="24.384" y2="43.2816" width="0.4064" layer="1"/>
-<wire x1="24.384" y1="47.3964" x2="24.4632" y2="47.5234" width="0.4064" layer="1"/>
+<wire x1="24.384" y1="49.3964" x2="24.4632" y2="47.5234" width="0.4064" layer="1"/>
 <wire x1="24.2316" y1="43.1292" x2="24.23" y2="42.98" width="0.4064" layer="1"/>
 <wire x1="34.29" y1="57.4548" x2="34.29" y2="57.912" width="0.4064" layer="1"/>

Commit message: 12
Parts:
- moved R43 1.00 mm to (76.2, 50.0)
Routing:
- net +5V: track 621.9 -> 622.8 mm
- net N$50: track 27.0 -> 27.9 mm
Changed lines of the file:
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@@
 <element name="R41" library="SparkFun-Resistors" package="1206" value="10k" x="84.074" y="50.2666"/>
 <element name="R40" library="SparkFun-Resistors" package="1206" value="2.2k" x="86.3854" y="64.5668" rot="R90"/>
-<element name="R43" library="SparkFun-Resistors" package="1206" value="10k" x="76.1746" y="50.9524" rot="R180"/>
+<element name="R43" library="SparkFun-Resistors" package="1206" value="10k" x="76.1746" y="49.9524" rot="R180"/>
 <element name="R44" library="SparkFun-Resistors" package="1206" value="10k" x="76.2254" y="46.863" rot="R180"/>
 <element name="R36" library="SparkFun-Resistors" package="1206" value="1k" x="85.1408" y="15.0876" rot="R180"/>
@@
 <wire x1="74.676" y1="55.1688" x2="74.676" y2="51.054" width="0.4064" layer="1"/>
 <wire x1="73.914" y1="56.5404" x2="74.676" y2="55.7784" width="0.4064" layer="1"/>
-<wire x1="74.676" y1="51.054" x2="74.7746" y2="50.9524" width="0.4064" layer="1"/>
+<wire x1="74.676" y1="51.054" x2="74.7746" y2="49.9524" width="0.4064" layer="1"/>
 <wire x1="73.914" y1="56.5404" x2="73.8454" y2="56.5948" width="0.4064" layer="1"/>
 <wire x1="96.4692" y1="49.8348" x2="96.4692" y2="53.6448" width="0.4064" layer="1"/>
@@
 <wire x1="77.5716" y1="46.7868" x2="77.6254" y2="46.863" width="0.4064" layer="1"/>
 <wire x1="77.5716" y1="46.9392" x2="77.5716" y2="50.9016" width="0.4064" layer="1"/>
-<wire x1="77.5716" y1="50.9016" x2="77.5746" y2="50.9524" width="0.4064" layer="1"/>
+<wire x1="77.5716" y1="50.9016" x2="77.5746" y2="49.9524" width="0.4064" layer="1"/>
 <wire x1="77.5716" y1="46.9392" x2="77.6254" y2="46.863" width="0.4064" layer="1"/>
 <wire x1="88.2396" y1="51.5112" x2="89.0016" y2="51.5112" width="0.4064" layer="1"/>
